File: KiCad/STM32H7_MCU.kicad_sch (KiCad schematic)
At the start: 53 parts, among them IC2 SN74LVC1G14DBVR, IC3 STM32H7R7L8H6H, IC4 TLV75718PDRVR, Y1 VXM7-9032-25M0000000

Commit message: BOM update
Parts:
- C11, C12, C15, C16, C18, C19, C25, C26, C28, C29, C30, C31, C32, C33, C34, C35, C36, C37, C38, C8, C9: DigiKey (none) -> 490-6287-1-ND; Mouser (none) -> 81-GRM155R60J104KA1D; TME (none) -> GRM155R60J104KA01D
- C22: DigiKey (none) -> 1276-6762-1-ND; LCSC (none) -> C472450; Mouser (none) -> 187-CL05C221JB51PNC; TME (none) -> CL05C221JB51PNC
- C6: DigiKey (none) -> 490-6309-1-ND; Mouser (none) -> 81-GRM155R61C103KA1D; TME (none) -> GRM155R61C103KA01D
- FB1: LCSC (none) -> C2661511
- L1: LCSC (none) -> C83998
- R1, R2: DigiKey (none) -> 311-1.50KLRCT-ND; LCSC (none) -> C114759; Mouser (none) -> 603-RC0402FR-071K5L; TME (none) -> RC0402FR-071K5L
- R3: DigiKey (none) -> 311-10.0KLRCT-ND; LCSC (none) -> C60490; Mouser (none) -> 603-RC0402FR-0710KL; TME (none) -> SMD0402-10K-1%
- R4, R5: DigiKey (none) -> 311-0.0LRCT-ND; LCSC (none) -> C106231; Mouser (none) -> 603-RC0402FR-070RL; TME (none) -> RC0402FR-070RL

Commit message: CEC and HPD signals fixed
Connections:
- net DVID_HPD: now reaches IC3.E11 (PE12)
- net TFT_DVID_CEC renamed DVID_CEC
- no-connect marks 26 -> 27
Changed lines of the file:
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@@
 	)
 	(no_connect
+		(at 149.86 30.48)
+	)
+	(no_connect
 		(at 149.86 99.06)
 	)
@@
 	)
 	(no_connect
-		(at 73.66 101.6)
+		(at 71.12 38.1)
 	)
 	(no_connect
-		(at 71.12 38.1)
+		(at 149.86 33.02)
 	)
 	(no_connect
@@
 	(wire
 		(pts
-			(xy 73.66 101.6) (xy 71.12 101.6)
+			(xy 76.2 101.6) (xy 71.12 101.6)
 		)
 		(stroke
@@
 		)
 	)
-	(global_label "TFT_DVID_CEC"
+	(global_label "DVID_CEC"
 		(shape output)
 		(at 35.56 86.36 180)
@@
 		)
 		(property "Intersheetrefs" "${INTERSHEET_REFS}"
-			(at 24.9116 86.36 0)
+			(at 27.7055 86.36 0)
 			(effects
 				(font
@@
 				(hide yes)
 			)
+		)
+	)
+	(global_label "DVID_HPD"
+		(shape input)
+		(at 76.2 101.6 0)
+		(fields_autoplaced yes)
+		(effects
+			(font
+				(size 0.889 0.889)
+				(color 255 153 0 1)
+			)
+			(justify left)
+		)
+		(property "Intersheetrefs" "${INTERSHEET_REFS}"
+			(at 84.1815 101.6 0)
+			(effects
+				(font
+					(size 1.27 1.27)
+				)
+				(justify left)
+				(hide yes)
+			)
