File: KiCad/STM32H7_MCU.kicad_sch (KiCad schematic)
At the start: 51 parts, among them IC2 SN74LVC1G14DBVR, IC3 STM32H7R7L8H6H, IC4 TLV75718PDRVR, Y1 VXM7-9032-25M0000000

Commit message: #1, #2, #3
Parts:
- added R23: 10K, PCM_EEZ_passives:R_0402_1005Metric, symbol PCM_EEZ_passives:R-EU
Connections:
- net +3V3: now also R23.2
- net ~{RESET_OUT}: now also R23.1
- net WDG_IN renamed DIB_OE_SYNC
Other:
- moved on the sheet: R3
Changed lines of the file:
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@@
 	(title_block
 		(title "${project_name}")
-		(date "2025-11-28")
+		(date "2025-12-19")
 		(rev "${project_version}")
 		(company "${project_creator}")
@@
 	)
 	(junction
+		(at 175.26 55.88)
+		(diameter 0)
+		(color 0 0 0 0)
+	)
+	(junction
 		(at 248.92 101.6)
 		(diameter 0)
@@
 	(wire
 		(pts
+			(xy 170.18 55.88) (xy 175.26 55.88)
+		)
+		(stroke
+			(width 0)
+			(type default)
+		)
+	)
+	(wire
+		(pts
 			(xy 71.12 147.32) (xy 76.2 147.32)
 		)
@@
 	(wire
 		(pts
+			(xy 175.26 53.34) (xy 175.26 55.88)
+		)
+		(stroke
+			(width 0)
+			(type default)
+		)
+	)
+	(wire
+		(pts
 			(xy 35.56 119.38) (xy 40.64 119.38)
 		)
@@
 	(wire
 		(pts
+			(xy 152.4 71.12) (xy 152.4 73.66)
+		)
+		(stroke
+			(width 0)
+			(type default)
+		)
+	)
+	(wire
+		(pts
 			(xy 88.9 180.34) (xy 93.98 180.34)
 		)
@@
 	(wire
 		(pts
-			(xy 152.4 73.66) (xy 154.94 73.66)
+			(xy 152.4 71.12) (xy 154.94 71.12)
 		)
 		(stroke
@@
 	(wire
 		(pts
+			(xy 162.56 76.2) (xy 170.18 76.2)
+		)
+		(stroke
+			(width 0)
+			(type default)
+		)
+	)
+	(wire
+		(pts
 			(xy 35.56 45.72) (xy 40.64 45.72)
 		)
@@
 	(wire
 		(pts
+			(xy 175.26 55.88) (xy 180.34 55.88)
+		)
+		(stroke
+			(width 0)
+			(type default)
+		)
+	)
+	(wire
+		(pts
 			(xy 248.92 106.68) (xy 248.92 109.22)
 		)
@@
 	(wire
 		(pts
-			(xy 160.02 76.2) (xy 152.4 76.2)
-		)
-		(stroke
-			(width 0)
-			(type default)
-		)
-	)
-	(wire
-		(pts
 			(xy 259.08 127) (xy 254 127)
 		)
@@
 		)
 	)
-	(wire
-		(pts
-			(xy 177.8 55.88) (xy 180.34 55.88)
-		)
-		(stroke
-			(width 0)
-			(type default)
-		)
-	)
 	(polyline
 		(pts
@@
 	(wire
 		(pts
+			(xy 170.18 55.88) (xy 170.18 58.42)
+		)
+		(stroke
+			(width 0)
+			(type default)
+		)
+	)
+	(wire
+		(pts
 			(xy 76.2 101.6) (xy 71.12 101.6)
 		)
@@
 	(global_label "BOOT0"
 		(shape input)
-		(at 154.94 73.66 0)
+		(at 154.94 71.12 0)
 		(fields_autoplaced yes)
 		(effects
@@
 		)
 		(property "Intersheetrefs" "${INTERSHEET_REFS}"
-			(at 160.8472 73.66 0)
+			(at 160.8472 71.12 0)
 			(effects
 				(font
@@
 		)
 	)
-	(global_label "WDG_IN"
+	(global_label "DIB_OE_SYNC"
 		(shape output)
 		(at 116.84 35.56 180)
@@
 		)
 		(property "Intersheetrefs" "${INTERSHEET_REFS}"
-			(at 110.3825 35.56 0)
+			(at 106.4879 35.56 0)
 			(effects
 				(font
@@
 	(symbol
 		(lib_id "PCM_EEZ_passives:R-EU")
-		(at 165.1 76.2 270)
+		(at 157.48 76.2 270)
 		(mirror x)
 		(unit 1)
@@
 		(dnp no)
 		(property "Reference" "R3"
-			(at 165.1 74.93 90)
+			(at 157.48 74.93 90)
 			(effects
 				(font
@@
 		)
 		(property "Value" "10K"
-			(at 165.1 77.47 90)
+			(at 157.48 77.47 90)
 			(effects
 				(font
@@
 		)
 		(property "Footprint" "PCM_EEZ_passives:R_0402_1005Metric"
-			(at 165.1 76.2 0)
+			(at 157.48 76.2 0)
 			(effects
 				(font
@@
 		)
 		(property "Datasheet" ""
-			(at 165.1 76.2 0)
+			(at 157.48 76.2 0)
 			(effects
 				(font
@@
 		)
 		(property "Description" ""
-			(at 165.1 76.2 0)
+			(at 157.48 76.2 0)
 			(effects
 				(font
@@
 		)
 		(property "DigiKey" "311-10.0KLRCT-ND"
-			(at 165.1 76.2 0)
+			(at 157.48 76.2 0)
 			(effects
 				(font
@@
 		)
 		(property "Mouser" "603-RC0402FR-0710KL"
-			(at 165.1 76.2 0)
+			(at 157.48 76.2 0)
 			(effects
 				(font
@@
 		)
 		(property "TME" "SMD0402-10K-1%"
-			(at 165.1 76.2 0)
+			(at 157.48 76.2 0)
 			(effects
 				(font
@@
 		)
 		(property "LCSC" "C60490"
-			(at 165.1 76.2 0)
+			(at 157.48 76.2 0)
 			(effects
 				(font
@@
 		)
 		(property "Type" ""
-			(at 165.1 76.2 0)
+			(at 157.48 76.2 0)
 			(effects
 				(font
@@
 	)
 	(symbol
+		(lib_id "PCM_EEZ_passives:R-EU")
+		(at 170.18 63.5 0)
+		(unit 1)
+		(exclude_from_sim no)
+		(in_bom yes)
+		(on_board yes)
+		(dnp no)
+		(property "Reference" "R23"
+			(at 171.45 61.595 0)
+			(effects
+				(font
+					(size 1.27 1.27)
+				)
+				(justify left top)
+			)
+		)
+		(property "Value" "10K"
+			(at 171.45 63.5 0)
+			(effects
+				(font
+					(size 1.27 1.27)
+				)
+				(justify left top)
+			)
+		)
+		(property "Footprint" "PCM_EEZ_passives:R_0402_1005Metric"
+			(at 170.18 63.5 0)
+			(effects
+				(font
+					(size 1.27 1.27)
+				)
+				(hide yes)
+			)
+		)
+		(property "Datasheet" ""
+			(at 170.18 63.5 0)
+			(effects
+				(font
+					(size 1.27 1.27)
+				)
+				(hide yes)
+			)
+		)
+		(property "Description" ""
+			(at 170.18 63.5 0)
+			(effects
+				(font
+					(size 1.27 1.27)
+				)
+				(hide yes)
+			)
+		)
+		(property "DigiKey" "311-10.0KLRCT-ND"
+			(at 170.18 63.5 0)
+			(effects
+				(font
+					(size 1.27 1.27)
+				)
+				(hide yes)
+			)
+		)
+		(property "Mouser" "603-RC0402FR-0710KL"
+			(at 170.18 63.5 0)
+			(effects
+				(font
+					(size 1.27 1.27)
+				)
+				(hide yes)
+			)
+		)
+		(property "TME" "SMD0402-10K-1%"
+			(at 170.18 63.5 0)
+			(effects
+				(font
+					(size 1.27 1.27)
+				)
+				(hide yes)
+			)
+		)
+		(property "LCSC" "C60490"
+			(at 170.18 63.5 0)
+			(effects
+				(font
+					(size 1.27 1.27)
+				)
+				(hide yes)
+			)
+		)
+		(property "Type" ""
+			(at 170.18 63.5 0)
+			(effects
+				(font
+					(size 1.27 1.27)
+				)
+				(hide yes)
+			)
+		)
+		(pin "1"
+		)
+		(pin "2"
+		)
+		(instances
+			(project "BB3plus CM5 STM32H7 module"
+				(path "/1a4f0aea-3a69-423f-8790-3103cd0321c4/d7166dbe-caf3-45a8-82fe-1ff0a9696e25"
+					(reference "R23")
+					(unit 1)
+				)
+			)
+		)
+	)
+	(symbol
 		(lib_id "PCM_EEZ_passives:L_Ferrite Bead")
 		(at 182.88 55.88 270)
@@
 	(symbol
 		(lib_id "PCM_EEZ_symbols:+3V3")
-		(at 175.26 55.88 90)
-		(mirror x)
+		(at 175.26 50.8 0)
+		(mirror y)
 		(unit 1)
 		(exclude_from_sim no)
@@
 		(dnp no)
 		(property "Reference" "#+3V07"
-			(at 175.26 55.88 0)
+			(at 175.26 50.8 0)
 			(effects
 				(font
@@
 		)
 		(property "Value" "+3V3"
-			(at 174.625 55.88 90)
+			(at 175.26 50.165 0)
 			(effects
 				(font
 					(size 1.27 1.27)
 				)
-				(justify left)
+				(justify bottom)
 			)
 		)
 		(property "Footprint" ""
-			(at 175.26 55.88 0)
+			(at 175.26 50.8 0)
 			(effects
 				(font
@@
 		)
 		(property "Datasheet" ""
-			(at 175.26 55.88 0)
+			(at 175.26 50.8 0)
 			(effects
 				(font
@@
 		)
 		(property "Description" "Power symbol creates a global label with name \"+3V3\""
-			(at 175.26 55.88 0)
+			(at 175.26 50.8 0)
 			(effects
 				(font

Commit message: #4
Parts:
- renumbered R23 to R4
Changed lines of the file:
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@@
 	(title_block
 		(title "${project_name}")
-		(date "2025-12-19")
+		(date "2025-12-24")
 		(rev "${project_version}")
 		(company "${project_creator}")
@@
 		(on_board yes)
 		(dnp no)
-		(property "Reference" "#PWR010"
+		(property "Reference" "#PWR011"
 			(at 251.46 80.01 0)
 			(effects
@@
 			(project "BB3plus CM5 STM32H7 module"
 				(path "/1a4f0aea-3a69-423f-8790-3103cd0321c4/d7166dbe-caf3-45a8-82fe-1ff0a9696e25"
-					(reference "#PWR010")
+					(reference "#PWR011")
 					(unit 1)
 				)
@@
 		(on_board yes)
 		(dnp no)
-		(property "Reference" "#PWR011"
+		(property "Reference" "#PWR012"
 			(at 270.51 109.22 0)
 			(effects
@@
 			(project "BB3plus CM5 STM32H7 module"
 				(path "/1a4f0aea-3a69-423f-8790-3103cd0321c4/d7166dbe-caf3-45a8-82fe-1ff0a9696e25"
-					(reference "#PWR011")
+					(reference "#PWR012")
 					(unit 1)
 				)
@@
 		(on_board yes)
 		(dnp no)
-		(property "Reference" "R23"
+		(property "Reference" "R4"
 			(at 171.45 61.595 0)
 			(effects
@@
 			(project "BB3plus CM5 STM32H7 module"
 				(path "/1a4f0aea-3a69-423f-8790-3103cd0321c4/d7166dbe-caf3-45a8-82fe-1ff0a9696e25"
-					(reference "R23")
+					(reference "R4")
 					(unit 1)
 				)
@@
 		(on_board yes)
 		(dnp no)
-		(property "Reference" "#PWR012"
+		(property "Reference" "#PWR013"
 			(at 273.05 132.08 0)
 			(effects
@@
 			(project "BB3plus CM5 STM32H7 module"
 				(path "/1a4f0aea-3a69-423f-8790-3103cd0321c4/d7166dbe-caf3-45a8-82fe-1ff0a9696e25"
-					(reference "#PWR012")
+					(reference "#PWR013")
 					(unit 1)
 				)
@@
 		(on_board yes)
 		(dnp no)
-		(property "Reference" "#PWR09"
+		(property "Reference" "#PWR010"
 			(at 163.83 175.26 0)
 			(effects
@@
 			(project "BB3plus CM5 STM32H7 module"
 				(path "/1a4f0aea-3a69-423f-8790-3103cd0321c4/d7166dbe-caf3-45a8-82fe-1ff0a9696e25"
-					(reference "#PWR09")
+					(reference "#PWR010")
 					(unit 1)
 				)

Commit message: #9
Parts:
- renumbered C9 to C10, C10 to C11, C11 to C12, C12 to C13, C13 to C14, C14 to C15, C15 to C16, C16 to C17, C17 to C18, C18 to C19, C19 to C20, C20 to C21, C21 to C22, C22 to C23, C23 to C24, C24 to C25, C25 to C26, C26 to C27, C27 to C28, C28 to C29, C29 to C30, C30 to C31, C31 to C32, C32 to C33, C33 to C34, C34 to C35, C35 to C36, C36 to C37, C37 to C38, C38 to C39, C3 to C4, C39 to C40, C40 to C41, C41 to C42, C4 to C5, C5 to C6, C6 to C7, C7 to C8, C8 to C9, IC2 to IC3, IC3 to IC4, IC4 to IC5
Connections:
- net USB_FS_SEL: now reaches IC4.L14 (PD14)
- net MCU_USB_ID: now reaches IC4.B8 (PM9)
- net MCU_USB_VBUS: now reaches IC4.C9 (PM8)
- no-connect marks 25 -> 22
