File: KiCad/BB3plus CM5 STM32H7 module.kicad_pcb (KiCad board)
At the start: 6 copper layers, 55 x 40 mm, 134 parts, among them IC1 AZ1117CH2-3.3TRG1, IC10 MX25UM25645GXDI00-T, IC2 SN74LVC1G14DBVR, IC3 STM32H7R7L8H6H, IC4 TLV75718PDRVR, IC5 MX52LM04A11XVW, IC6 LAN8742A-CZ-TR, IC7 APS256XXN-OBR-BG, IC8 TFP410PAP, IC9 TS3DV642A0RUAR, Y1 VXM7-9032-25M0000000, Y2 VXM7-9032-25M0000000

Commit message: #1, #2, #3
Parts:
- added JP2: ~, PCM_EEZ_SMD:JP2 shorted (0603), B.Cu at (117.8, 77.9)
- added R23: 10K, PCM_EEZ_passives:R_0402_1005Metric, F.Cu at (122.3, 102.0)
- IC10: footprint PCM_EEZ_BGA:BGA24C100P5X5_800X600X120 -> PCM_EEZ_BGA:APS256XXN-OBR-BG_APY-L
- R21: moved to F.Cu
- moved R22 10.5 mm to (110.5, 78.4), turned to 90 degrees
- moved R21 5.25 mm to (114.7, 84.7)
- moved C73 5.06 mm to (115.5, 80.2), turned to -90 degrees
- moved C72 3.24 mm to (114.3, 80.7), turned to -90 degrees
- moved C75 1.07 mm to (119.1, 81.2)
- moved C74 1.07 mm to (118.6, 80.0)
- moved C76 0.73 mm to (115.6, 84.1)
- moved C77 0.73 mm to (116.8, 84.7)
- moved IC10 0.08 mm to (115.3, 80.9), turned to 90 degrees
Connections:
- net WDG_IN renamed DIB_OE_SYNC
- SoM1 pad 111: unconnected-(SoM1B-VBUS_EN_(3.3v)-Pad111) -> Net-(SoM1B-VBUS_EN_(3.3v))
Routing:
- net ~{RESET_OUT}: track 110.8 -> 113.5 mm
- net ~{XSPIM_P2_CS1}: track 15.8 -> 13.4 mm, vias 1 -> 0
- net XSPIM_P2_IO7: track 13.5 -> 11.3 mm
- net XSPIM_P2_IO2: track 13.4 -> 15.2 mm
- net +3V3: track 33.2 -> 34.9 mm
- net RS485_TX/DOUT3: track 53.0 -> 51.3 mm
- net +1V8: track 40.1 -> 41.8 mm, vias 24 -> 26
- net XSPIM_P2_IO0: track 13.9 -> 12.3 mm
- net XSPIM_P2_IO5: track 13.4 -> 15.0 mm
- net Net-(SoM1B-VBUS_EN_(3.3v)): track 0.00 -> 1.55 mm
- net XSPIM_P2_IO3: track 13.5 -> 15.0 mm
- net DIB1_USB_D+: track 31.9 -> 33.4 mm
- net XSPIM_P2_DQS0: track 10.9 -> 12.2 mm
- net XSPIM_P2_CLK: track 13.3 -> 12.0 mm, vias 0 -> 2
- net XSPIM_P2_IO6: track 13.3 -> 14.7 mm
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
Commit message: #4
Parts:
- IC5: value MX52LM04A11XVW -> IS21EF04GP-JQLI; footprint PCM_EEZ_BGA:BGA153_MX52LM_EMMC -> PCM_EEZ_BGA:IS21EF04GP-JQLI
- moved C3 49.6 mm to (140.5, 106.4), turned to -90 degrees
- moved IC4 47.0 mm to (138.8, 106.8), turned to 0 degrees
- moved C6 44.6 mm to (137.1, 107.2), turned to -90 degrees
- moved FM1 8.14 mm to (95.5, 79.0)
- moved C47 6.11 mm to (97.6, 87.1), turned to -90 degrees
- moved C44 5.85 mm to (96.7, 87.1), turned to -90 degrees
- moved C45 5.64 mm to (104.0, 88.5), turned to 90 degrees
- moved C46 5.30 mm to (101.3, 84.5)
- moved C49 5.30 mm to (100.4, 84.5)
- moved C48 4.66 mm to (103.1, 88.5), turned to 90 degrees
- moved C55 3.51 mm to (98.7, 100.7), turned to -90 degrees
- moved LOGO5 2.65 mm to (118.8, 75.1)
- moved R23 2.36 mm to (112.0, 76.6)
- moved X1 2.09 mm to (105.8, 76.3), turned to 180 degrees
- moved LOGO1 2.06 mm to (128.3, 76.0)
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- renumbered JP2 to JP1, JP1 to JP2, R9 to R10, R10 to R11, R11 to R12, R12 to R13, R13 to R14, R14 to R15, R15 to R16, R16 to R17, R17 to R18, R18 to R19, R19 to R20, R20 to R21, R21 to R22, R22 to R23, R23 to R4, R4 to R5, R5 to R6, R6 to R7, R7 to R8, R8 to R9
Connections:
- IC5 pad G3: unconnected-(IC5-RFU-PadG3) -> GND
- IC5 pad K5: ~{RESET_OUT} -> unconnected-(IC5-DS-PadK5)
- IC5 pad K8: GND -> SDMMC_D5
- IC5 pad K9: +3V3 -> SDMMC_D7
- IC5 pad M4: +1V8 -> GND
- IC5 pad M5: SDMMC_CMD -> ~{RESET_OUT}
- IC5 pad N2: GND -> SDMMC_D1
- IC5 pad P5: +1V8 -> SDMMC_CMD
- IC5 pad P6: GND -> SDMMC_CLK
Routing:
- net GND: track 100.4 -> 109.6 mm, vias 238 -> 237
- net +3V3: track 34.9 -> 43.4 mm, vias 46 -> 44
- net +1V8: track 41.8 -> 35.7 mm, vias 26 -> 35
- net SDMMC_D2: track 17.2 -> 22.7 mm
- net SDMMC_D1: track 17.2 -> 22.4 mm
- net SDMMC_D3: track 17.6 -> 22.3 mm
- net SDMMC_D7: track 17.6 -> 13.1 mm
- net SDMMC_D0: track 17.3 -> 21.2 mm
- net ~{RESET_OUT}: track 113.5 -> 117.4 mm
- net SDMMC_D4: track 17.5 -> 21.1 mm
- net SDMMC_D6: track 17.7 -> 21.2 mm
- net SDMMC_D5: track 17.6 -> 21.0 mm
- net /STM32H7 MCU/JTAG_SWDIO: track 18.1 -> 20.6 mm
- net SDMMC_CMD: track 17.3 -> 15.0 mm
- net SDMMC_CLK: track 17.7 -> 15.9 mm
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
Commit message: #6
Connections:
- IC8 pad 36: LTDC_G7 -> LTDC_R7
- IC8 pad 37: LTDC_G6 -> LTDC_R6
- IC8 pad 38: LTDC_G5 -> LTDC_R5
- IC8 pad 39: LTDC_G4 -> LTDC_R4
- IC8 pad 44: LTDC_R7 -> LTDC_G7
- IC8 pad 45: LTDC_R6 -> LTDC_G6
- IC8 pad 46: LTDC_R5 -> LTDC_G5
- IC8 pad 47: LTDC_R4 -> LTDC_G4
Routing:
- net LTDC_R7: track 34.7 -> 29.5 mm
- net LTDC_R5: track 32.1 -> 27.1 mm
- net LTDC_R6: track 33.5 -> 28.8 mm
- net LTDC_G7: track 19.4 -> 24.0 mm
- net LTDC_R4: track 38.9 -> 34.3 mm
- net LTDC_G6: track 19.1 -> 23.6 mm, vias 2 -> 0
- net LTDC_G5: track 21.4 -> 25.6 mm
- net LTDC_G4: track 20.5 -> 24.3 mm, vias 2 -> 0
- net ~{RESET_OUT}: track 117.4 -> 119.0 mm
- net GND: track 109.6 -> 110.3 mm
