File: KiCad/BB3plus CM5 STM32H7 module.kicad_pcb (KiCad board)
At the start: 6 copper layers, 55 x 40 mm, 136 parts, among them IC1 AZ1117CH2-3.3TRG1, IC10 MX25UM25645GXDI00-T, IC2 SN74LVC1G14DBVR, IC3 STM32H7R7L8H6H, IC4 TLV75718PDRVR, IC5 IS21EF04GP-JQLI, IC6 LAN8742A-CZ-TR, IC7 APS256XXN-OBR-BG, IC8 TFP410PAP, IC9 TS3DV642A0RUAR, Y1 VXM7-9032-25M0000000, Y2 VXM7-9032-25M0000000

Commit message: #7
Parts:
- added C72: 100n, PCM_EEZ_passives:C_0402_1005Metric, F.Cu at (135.6, 74.0)
- added C73: 100n, PCM_EEZ_passives:C_0402_1005Metric, F.Cu at (140.3, 74.0)
- added IC10: LSF0102DCH, PCM_EEZ_SMD:U_SOT765-1_NEX-L, F.Cu at (137.9, 75.1)
- renumbered C72 to C74, C73 to C75, C74 to C76, C75 to C77, C76 to C78, C77 to C79, IC10 to IC11
Connections:
- net /CM5 socket/+5V_IN renamed +5V
- IC9 pad 39: REAR_DVID_SDA -> Net-(IC10-A2)
- IC9 pad 40: REAR_DVID_SCL -> Net-(IC10-A1)
Routing:
- net +5V: track 0.00 -> 31.9 mm, vias 10 -> 11
- net Net-(IC10-A1): track 0.00 -> 23.4 mm
- net Net-(IC10-A2): track 0.00 -> 22.4 mm
- net REAR_DVID_SCL: track 21.5 -> 6.35 mm
- net REAR_DVID_SDA: track 16.9 -> 6.52 mm, vias 2 -> 1
- net +3V3: track 43.6 -> 48.2 mm, vias 44 -> 45
- net REAR_DVID_CEC: track 12.7 -> 11.0 mm, vias 2 -> 1
- net ~{RESET_OUT}: track 119.0 -> 118.3 mm
- net GND: track 110.3 -> 110.5 mm, vias 237 -> 240
- net REAR_DVID_HPD: track 9.69 -> 9.87 mm, vias 2 -> 1

Commit message: #8
Parts:
- added R23: 1K5, PCM_EEZ_passives:R_0402_1005Metric, F.Cu at (140.0, 75.0)
- added R24: 1K5, PCM_EEZ_passives:R_0402_1005Metric, F.Cu at (140.0, 76.0)
- IC10: value LSF0102DCH -> LSF0204GU12; footprint PCM_EEZ_SMD:U_SOT765-1_NEX-L -> PCM_EEZ_SMD:XQFN12_SOT1174-1_NEX-L
- moved C73 0.75 mm to (139.6, 73.7)
- moved C72 0.46 mm to (135.9, 73.7)
- moved IC10 0.21 mm to (137.7, 75.2)
- renumbered R23 to R25
Connections:
- IC10 pad 1: GND -> +3V3
- IC10 pad 2: +3V3 -> Net-(IC10-A1)
- IC10 pad 3: Net-(IC10-A1) -> Net-(IC10-A2)
- IC10 pad 4: Net-(IC10-A2) -> Net-(IC10-A3)
- IC10 pad 5: REAR_DVID_SDA -> Net-(IC10-A4)
- IC10 pad 6: REAR_DVID_SCL -> GND
- IC10 pad 7: +5V -> REAR_DVID_CEC
- IC10 pad 8: +3V3 -> REAR_DVID_HPD
- IC9 pad 20: REAR_DVID_CEC -> Net-(IC10-A4)
- IC9 pad 21: REAR_DVID_HPD -> Net-(IC10-A3)
Routing:
- net Net-(IC10-A4): track 0.00 -> 8.96 mm
- net Net-(IC10-A3): track 0.00 -> 8.76 mm
- net REAR_DVID_HPD: track 9.87 -> 17.1 mm
- net REAR_DVID_CEC: track 11.0 -> 16.3 mm
- net +5V: track 31.9 -> 34.6 mm
- net REAR_DVID_SDA: track 6.52 -> 8.55 mm
- net +3V3: track 48.2 -> 47.5 mm
