File: KiCad/Ethernet_flash.kicad_sch (KiCad schematic)
At the start: 30 parts, among them IC10 MX25UM25645GXDI00-T, IC8 TFP410PAP, IC9 TS3DV642A0RUAR

Commit message: #1, #2, #3
Parts:
- IC10: footprint PCM_EEZ_BGA:BGA24C100P5X5_800X600X120 -> PCM_EEZ_BGA:APS256XXN-OBR-BG_APY-L
Changed lines of the file:
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@@
 	(title_block
 		(title "${project_name}")
-		(date "2025-11-28")
+		(date "2025-12-19")
 		(rev "${project_version}")
 		(company "${project_creator}")
@@
 			)
 		)
-		(property "Footprint" "PCM_EEZ_BGA:BGA24C100P5X5_800X600X120"
+		(property "Footprint" "PCM_EEZ_BGA:APS256XXN-OBR-BG_APY-L"
 			(at 208.28 88.9 0)
 			(effects

Commit message: #4
Parts:
- renumbered JP1 to JP2, R17 to R18, R18 to R19, R19 to R20, R20 to R21, R21 to R22, R22 to R23
Changed lines of the file:
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@@
 	(title_block
 		(title "${project_name}")
-		(date "2025-12-19")
+		(date "2025-12-24")
 		(rev "${project_version}")
 		(company "${project_creator}")
@@
 		(on_board yes)
 		(dnp no)
-		(property "Reference" "#SUPPLY042"
+		(property "Reference" "#SUPPLY043"
 			(at 279.4 43.18 0)
 			(effects
@@
 			(project "BB3plus CM5 STM32H7 module"
 				(path "/1a4f0aea-3a69-423f-8790-3103cd0321c4/6c545e17-ca5e-4b04-9dff-4169dbe59c9e"
-					(reference "#SUPPLY042")
+					(reference "#SUPPLY043")
 					(unit 1)
 				)
@@
 		(on_board yes)
 		(dnp no)
-		(property "Reference" "#PWR016"
+		(property "Reference" "#PWR017"
 			(at 203.2 29.21 0)
 			(effects
@@
 			(project "BB3plus CM5 STM32H7 module"
 				(path "/1a4f0aea-3a69-423f-8790-3103cd0321c4/6c545e17-ca5e-4b04-9dff-4169dbe59c9e"
-					(reference "#PWR016")
+					(reference "#PWR017")
 					(unit 1)
 				)
@@
 		(on_board yes)
 		(dnp no)
-		(property "Reference" "#FLG06"
+		(property "Reference" "#FLG05"
 			(at 68.58 97.155 0)
 			(effects
@@
 			(project "BB3plus CM5 STM32H7 module"
 				(path "/1a4f0aea-3a69-423f-8790-3103cd0321c4/6c545e17-ca5e-4b04-9dff-4169dbe59c9e"
-					(reference "#FLG06")
+					(reference "#FLG05")
 					(unit 1)
 				)
@@
 		(on_board yes)
 		(dnp no)
-		(property "Reference" "#SUPPLY035"
+		(property "Reference" "#SUPPLY036"
 			(at 66.04 83.82 0)
 			(effects
@@
 			(project "BB3plus CM5 STM32H7 module"
 				(path "/1a4f0aea-3a69-423f-8790-3103cd0321c4/6c545e17-ca5e-4b04-9dff-4169dbe59c9e"
-					(reference "#SUPPLY035")
+					(reference "#SUPPLY036")
 					(unit 1)
 				)
@@
 		(on_board yes)
 		(dnp no)
-		(property "Reference" "R19"
+		(property "Reference" "R20"
 			(at 67.31 78.105 0)
 			(effects
@@
 			(project "BB3plus CM5 STM32H7 module"
 				(path "/1a4f0aea-3a69-423f-8790-3103cd0321c4/6c545e17-ca5e-4b04-9dff-4169dbe59c9e"
-					(reference "R19")
+					(reference "R20")
 					(unit 1)
 				)
@@
 		(on_board yes)
 		(dnp no)
-		(property "Reference" "R18"
+		(property "Reference" "R19"
 			(at 30.48 57.15 90)
 			(effects
@@
 			(project "BB3plus CM5 STM32H7 module"
 				(path "/1a4f0aea-3a69-423f-8790-3103cd0321c4/6c545e17-ca5e-4b04-9dff-4169dbe59c9e"
-					(reference "R18")
+					(reference "R19")
 					(unit 1)
 				)
@@
 		(on_board yes)
 		(dnp no)
-		(property "Reference" "R20"
+		(property "Reference" "R21"
 			(at 71.12 90.17 90)
 			(effects
@@
 			(project "BB3plus CM5 STM32H7 module"
 				(path "/1a4f0aea-3a69-423f-8790-3103cd0321c4/6c545e17-ca5e-4b04-9dff-4169dbe59c9e"
-					(reference "R20")
+					(reference "R21")
 					(unit 1)
 				)
@@
 		(on_board yes)
 		(dnp no)
-		(property "Reference" "R21"
+		(property "Reference" "R22"
 			(at 204.47 33.655 0)
 			(effects
@@
 			(project "BB3plus CM5 STM32H7 module"
 				(path "/1a4f0aea-3a69-423f-8790-3103cd0321c4/6c545e17-ca5e-4b04-9dff-4169dbe59c9e"
-					(reference "R21")
+					(reference "R22")
 					(unit 1)
 				)
@@
 		(on_board yes)
 		(dnp no)
-		(property "Reference" "#SUPPLY033"
+		(property "Reference" "#SUPPLY034"
 			(at 33.02 149.86 0)
 			(effects
@@
 			(project "BB3plus CM5 STM32H7 module"
 				(path "/1a4f0aea-3a69-423f-8790-3103cd0321c4/6c545e17-ca5e-4b04-9dff-4169dbe59c9e"
-					(reference "#SUPPLY033")
+					(reference "#SUPPLY034")
 					(unit 1)
 				)
@@
 		(on_board yes)
 		(dnp no)
-		(property "Reference" "#SUPPLY031"
+		(property "Reference" "#SUPPLY032"
 			(at 22.86 154.94 0)
 			(effects
@@
 			(project "BB3plus CM5 STM32H7 module"
 				(path "/1a4f0aea-3a69-423f-8790-3103cd0321c4/6c545e17-ca5e-4b04-9dff-4169dbe59c9e"
-					(reference "#SUPPLY031")
+					(reference "#SUPPLY032")
 					(unit 1)
 				)
@@
 		(on_board yes)
 		(dnp no)
-		(property "Reference" "#SUPPLY036"
+		(property "Reference" "#SUPPLY037"
 			(at 86.36 106.68 0)
 			(effects
@@
 			(project "BB3plus CM5 STM32H7 module"
 				(path "/1a4f0aea-3a69-423f-8790-3103cd0321c4/6c545e17-ca5e-4b04-9dff-4169dbe59c9e"
-					(reference "#SUPPLY036")
+					(reference "#SUPPLY037")
 					(unit 1)
 				)
@@
 		(on_board yes)
 		(dnp no)
-		(property "Reference" "#SUPPLY037"
+		(property "Reference" "#SUPPLY038"
 			(at 86.36 119.38 0)
 			(effects
@@
 			(project "BB3plus CM5 STM32H7 module"
 				(path "/1a4f0aea-3a69-423f-8790-3103cd0321c4/6c545e17-ca5e-4b04-9dff-4169dbe59c9e"
-					(reference "#SUPPLY037")
+					(reference "#SUPPLY038")
 					(unit 1)
 				)
@@
 		(on_board yes)
 		(dnp no)
-		(property "Reference" "#SUPPLY039"
+		(property "Reference" "#SUPPLY040"
 			(at 160.02 119.38 0)
 			(effects
@@
 			(project "BB3plus CM5 STM32H7 module"
 				(path "/1a4f0aea-3a69-423f-8790-3103cd0321c4/6c545e17-ca5e-4b04-9dff-4169dbe59c9e"
-					(reference "#SUPPLY039")
+					(reference "#SUPPLY040")
 					(unit 1)
 				)
@@
 		(on_board yes)
 		(dnp no)
-		(property "Reference" "#PWR017"
+		(property "Reference" "#PWR018"
 			(at 256.54 52.07 0)
 			(effects
@@
 			(project "BB3plus CM5 STM32H7 module"
 				(path "/1a4f0aea-3a69-423f-8790-3103cd0321c4/6c545e17-ca5e-4b04-9dff-4169dbe59c9e"
-					(reference "#PWR017")
+					(reference "#PWR018")
 					(unit 1)
 				)
@@
 		(on_board yes)
 		(dnp no)
-		(property "Reference" "#SUPPLY032"
+		(property "Reference" "#SUPPLY033"
 			(at 30.48 45.72 0)
 			(effects
@@
 			(project "BB3plus CM5 STM32H7 module"
 				(path "/1a4f0aea-3a69-423f-8790-3103cd0321c4/6c545e17-ca5e-4b04-9dff-4169dbe59c9e"
-					(reference "#SUPPLY032")
+					(reference "#SUPPLY033")
 					(unit 1)
 				)
@@
 		(on_board yes)
 		(dnp no)
-		(property "Reference" "#SUPPLY040"
+		(property "Reference" "#SUPPLY041"
 			(at 170.18 119.38 0)
 			(effects
@@
 			(project "BB3plus CM5 STM32H7 module"
 				(path "/1a4f0aea-3a69-423f-8790-3103cd0321c4/6c545e17-ca5e-4b04-9dff-4169dbe59c9e"
-					(reference "#SUPPLY040")
+					(reference "#SUPPLY041")
 					(unit 1)
 				)
@@
 		(on_board yes)
 		(dnp no)
-		(property "Reference" "#FLG08"
+		(property "Reference" "#FLG07"
 			(at 78.74 122.555 0)
 			(effects
@@
 			(project "BB3plus CM5 STM32H7 module"
 				(path "/1a4f0aea-3a69-423f-8790-3103cd0321c4/6c545e17-ca5e-4b04-9dff-4169dbe59c9e"
-					(reference "#FLG08")
+					(reference "#FLG07")
 					(unit 1)
 				)
@@
 		(on_board yes)
 		(dnp no)
-		(property "Reference" "#SUPPLY038"
+		(property "Reference" "#SUPPLY039"
 			(at 86.36 132.08 0)
 			(effects
@@
 			(project "BB3plus CM5 STM32H7 module"
 				(path "/1a4f0aea-3a69-423f-8790-3103cd0321c4/6c545e17-ca5e-4b04-9dff-4169dbe59c9e"
-					(reference "#SUPPLY038")
+					(reference "#SUPPLY039")
 					(unit 1)
 				)
@@
 		(on_board yes)
 		(dnp no)
-		(property "Reference" "#SUPPLY041"
+		(property "Reference" "#SUPPLY042"
 			(at 246.38 55.88 0)
 			(effects
@@
 			(project "BB3plus CM5 STM32H7 module"
 				(path "/1a4f0aea-3a69-423f-8790-3103cd0321c4/6c545e17-ca5e-4b04-9dff-4169dbe59c9e"
-					(reference "#SUPPLY041")
+					(reference "#SUPPLY042")
 					(unit 1)
 				)
@@
 		(on_board yes)
 		(dnp no)
-		(property "Reference" "R22"
+		(property "Reference" "R23"
 			(at 257.81 53.975 0)
 			(effects
@@
 			(project "BB3plus CM5 STM32H7 module"
 				(path "/1a4f0aea-3a69-423f-8790-3103cd0321c4/6c545e17-ca5e-4b04-9dff-4169dbe59c9e"
-					(reference "R22")
+					(reference "R23")
 					(unit 1)
 				)
@@
 		(on_board yes)
 		(dnp no)
-		(property "Reference" "#PWR018"
+		(property "Reference" "#PWR019"
 			(at 279.4 34.29 0)
 			(effects
@@
 			(project "BB3plus CM5 STM32H7 module"
 				(path "/1a4f0aea-3a69-423f-8790-3103cd0321c4/6c545e17-ca5e-4b04-9dff-4169dbe59c9e"
-					(reference "#PWR018")
+					(reference "#PWR019")
 					(unit 1)
 				)
@@
 		(on_board yes)
 		(dnp no)
-		(property "Reference" "R17"
+		(property "Reference" "R18"
 			(at 27.94 123.19 90)
 			(effects
@@
 			(project "BB3plus CM5 STM32H7 module"
 				(path "/1a4f0aea-3a69-423f-8790-3103cd0321c4/6c545e17-ca5e-4b04-9dff-4169dbe59c9e"
-					(reference "R17")
+					(reference "R18")
 					(unit 1)
 				)
@@
 		(on_board yes)
 		(dnp no)
-		(property "Reference" "#FLG07"
+		(property "Reference" "#FLG06"
 			(at 68.58 109.855 0)
 			(effects
@@
 			(project "BB3plus CM5 STM32H7 module"
 				(path "/1a4f0aea-3a69-423f-8790-3103cd0321c4/6c545e17-ca5e-4b04-9dff-4169dbe59c9e"
-					(reference "#FLG07")
+					(reference "#FLG06")
 					(unit 1)
 				)
@@
 		(on_board yes)
 		(dnp no)
-		(property "Reference" "#SUPPLY034"
+		(property "Reference" "#SUPPLY035"
 			(at 63.5 149.86 0)
 			(effects
@@
 			(project "BB3plus CM5 STM32H7 module"
 				(path "/1a4f0aea-3a69-423f-8790-3103cd0321c4/6c545e17-ca5e-4b04-9dff-4169dbe59c9e"
-					(reference "#SUPPLY034")
+					(reference "#SUPPLY035")
 					(unit 1)
 				)
@@
 		(on_board yes)
 		(dnp no)
-		(property "Reference" "JP1"
+		(property "Reference" "JP2"
 			(at 21.59 147.3199 0)
 			(effects
@@
 			(project "BB3plus CM5 STM32H7 module"
 				(path "/1a4f0aea-3a69-423f-8790-3103cd0321c4/6c545e17-ca5e-4b04-9dff-4169dbe59c9e"
-					(reference "JP1")
+					(reference "JP2")
 					(unit 1)
 				)

Commit message: #6
Connections:
- net LTDC_G4: now also IC8.47 (DATA12); no longer IC8.39 (DATA20)
- net LTDC_G5: now also IC8.46 (DATA13); no longer IC8.38 (DATA21)
- net LTDC_G6: now also IC8.45 (DATA14); no longer IC8.37 (DATA22)
- net LTDC_G7: now also IC8.44 (DATA15); no longer IC8.36 (DATA23)
- net LTDC_R4: now also IC8.39 (DATA20); no longer IC8.47 (DATA12)
- net LTDC_R5: now also IC8.38 (DATA21); no longer IC8.46 (DATA13)
- net LTDC_R6: now also IC8.37 (DATA22); no longer IC8.45 (DATA14)
- net LTDC_R7: now also IC8.36 (DATA23); no longer IC8.44 (DATA15)
Changed lines of the file:
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@@
 	(title_block
 		(title "${project_name}")
-		(date "2025-12-24")
+		(date "2025-12-27")
 		(rev "${project_version}")
 		(company "${project_creator}")
@@
 	)
 	(junction
-		(at 33.02 139.7)
-		(diameter 0)
-		(color 0 0 0 0)
-	)
-	(junction
 		(at 73.66 99.06)
 		(diameter 0)
@@
 		(color 0 0 0 0)
 	)
+	(junction
+		(at 33.02 139.7)
+		(diameter 0)
+		(color 0 0 0 0)
+	)
 	(no_connect
 		(at 241.3 68.58)
@@
 	(wire
 		(pts
-			(xy 27.94 116.84) (xy 35.56 116.84)
-		)
-		(stroke
-			(width 0)
-			(type default)
-		)
-	)
-	(wire
-		(pts
 			(xy 22.86 142.24) (xy 22.86 144.78)
 		)
@@
 	(wire
 		(pts
-			(xy 27.94 114.3) (xy 35.56 114.3)
+			(xy 63.5 127) (xy 63.5 129.54)
 		)
 		(stroke
@@
 	(wire
 		(pts
-			(xy 63.5 127) (xy 63.5 129.54)
+			(xy 30.48 43.18) (xy 30.48 45.72)
 		)
 		(stroke
@@
 	(wire
 		(pts
-			(xy 30.48 43.18) (xy 30.48 45.72)
+			(xy 22.86 127) (xy 35.56 127)
 		)
 		(stroke
@@
 	(wire
 		(pts
-			(xy 22.86 127) (xy 35.56 127)
+			(xy 203.2 40.64) (xy 208.28 40.64)
 		)
 		(stroke
@@
 	(wire
 		(pts
-			(xy 203.2 40.64) (xy 208.28 40.64)
+			(xy 27.94 119.38) (xy 35.56 119.38)
 		)
 		(stroke
@@
 	(wire
 		(pts
-			(xy 27.94 96.52) (xy 35.56 96.52)
-		)
-		(stroke
-			(width 0)
-			(type default)
-		)
-	)
-	(wire
-		(pts
 			(xy 86.36 119.38) (xy 68.58 119.38)
 		)
@@
 	(wire
 		(pts
+			(xy 27.94 111.76) (xy 35.56 111.76)
+		)
+		(stroke
+			(width 0)
+			(type default)
+		)
+	)
+	(wire
+		(pts
 			(xy 243.84 53.34) (xy 243.84 55.88)
 		)
@@
 	(wire
 		(pts
-			(xy 33.02 134.62) (xy 35.56 134.62)
-		)
-		(stroke
-			(width 0)
-			(type default)
-		)
-	)
-	(wire
-		(pts
 			(xy 63.5 142.24) (xy 63.5 144.78)
 		)
@@
 	(wire
 		(pts
-			(xy 27.94 111.76) (xy 35.56 111.76)
+			(xy 241.3 53.34) (xy 243.84 53.34)
 		)
 		(stroke
@@
 	(wire
 		(pts
-			(xy 241.3 53.34) (xy 243.84 53.34)
+			(xy 160.02 116.84) (xy 160.02 119.38)
 		)
 		(stroke
@@
 	(wire
 		(pts
-			(xy 160.02 116.84) (xy 160.02 119.38)
+			(xy 60.96 40.64) (xy 68.58 40.64)
 		)
 		(stroke
@@
 	(wire
 		(pts
-			(xy 60.96 40.64) (xy 68.58 40.64)
+			(xy 33.02 134.62) (xy 33.02 139.7)
 		)
 		(stroke
@@
 	(wire
 		(pts
-			(xy 27.94 119.38) (xy 35.56 119.38)
-		)
-		(stroke
-			(width 0)
-			(type default)
-		)
-	)
-	(wire
-		(pts
 			(xy 63.5 139.7) (xy 63.5 142.24)
 		)
@@
 	(wire
 		(pts
+			(xy 27.94 91.44) (xy 35.56 91.44)
+		)
+		(stroke
+			(width 0)
+			(type default)
+		)
+	)
+	(wire
+		(pts
 			(xy 116.84 55.88) (xy 124.46 55.88)
 		)
@@
 	(wire
 		(pts
-			(xy 27.94 99.06) (xy 35.56 99.06)
-		)
-		(stroke
-			(width 0)
-			(type default)
-		)
-	)
-	(wire
-		(pts
 			(xy 63.5 111.76) (xy 63.5 114.3)
 		)
@@
 	(wire
 		(pts
+			(xy 27.94 114.3) (xy 35.56 114.3)
+		)
+		(stroke
+			(width 0)
+			(type default)
+		)
+	)
+	(wire
+		(pts
 			(xy 60.96 147.32) (xy 63.5 147.32)
 		)
@@
 	(wire
 		(pts
+			(xy 27.94 116.84) (xy 35.56 116.84)
+		)
+		(stroke
+			(width 0)
+			(type default)
+		)
+	)
+	(wire
+		(pts
 			(xy 101.6 99.06) (xy 104.14 99.06)
 		)
@@
 	(wire
 		(pts
-			(xy 27.94 91.44) (xy 35.56 91.44)
+			(xy 121.92 93.98) (xy 124.46 93.98)
 		)
 		(stroke
@@
 	(wire
 		(pts
-			(xy 121.92 93.98) (xy 124.46 93.98)
+			(xy 27.94 71.12) (xy 35.56 71.12)
 		)
 		(stroke
@@
 	(wire
 		(pts
-			(xy 27.94 71.12) (xy 35.56 71.12)
+			(xy 116.84 71.12) (xy 124.46 71.12)
 		)
 		(stroke
@@
 	(wire
 		(pts
-			(xy 116.84 71.12) (xy 124.46 71.12)
+			(xy 33.02 144.78) (xy 33.02 147.32)
 		)
 		(stroke
@@
 	(wire
 		(pts
-			(xy 33.02 144.78) (xy 33.02 147.32)
+			(xy 63.5 144.78) (xy 63.5 147.32)
 		)
 		(stroke
@@
 	(wire
 		(pts
-			(xy 63.5 144.78) (xy 63.5 147.32)
+			(xy 200.66 50.8) (xy 208.28 50.8)
 		)
 		(stroke
@@
 	(wire
 		(pts
-			(xy 200.66 50.8) (xy 208.28 50.8)
+			(xy 27.94 96.52) (xy 35.56 96.52)
 		)
 		(stroke
@@
 	(wire
 		(pts
+			(xy 33.02 134.62) (xy 35.56 134.62)
+		)
+		(stroke
+			(width 0)
+			(type default)
+		)
+	)
+	(wire
+		(pts
 			(xy 157.48 111.76) (xy 165.1 111.76)
 		)
@@
 	(wire
 		(pts
-			(xy 200.66 73.66) (xy 208.28 73.66)
+			(xy 27.94 99.06) (xy 35.56 99.06)
 		)
 		(stroke
@@
 	(wire
 		(pts
-			(xy 63.5 99.06) (xy 68.58 99.06)
+			(xy 200.66 73.66) (xy 208.28 73.66)
 		)
 		(stroke
@@
 	(wire
 		(pts
-			(xy 33.02 134.62) (xy 33.02 139.7)
+			(xy 63.5 99.06) (xy 68.58 99.06)
 		)
 		(stroke
@@
 	(global_label "LTDC_R4"
 		(shape input)
-		(at 27.94 91.44 180)
+		(at 27.94 111.76 180)
 		(fields_autoplaced yes)
 		(effects
@@
 		)
 		(property "Intersheetrefs" "${INTERSHEET_REFS}"
-			(at 20.7204 91.44 0)
+			(at 20.7204 111.76 0)
 			(effects
 				(font
@@
 	(global_label "LTDC_R5"
 		(shape input)
-		(at 27.94 93.98 180)
+		(at 27.94 114.3 180)
 		(fields_autoplaced yes)
 		(effects
@@
 		)
 		(property "Intersheetrefs" "${INTERSHEET_REFS}"
-			(at 20.7204 93.98 0)
+			(at 20.7204 114.3 0)
 			(effects
 				(font
@@
 	(global_label "LTDC_G6"
 		(shape input)
-		(at 27.94 116.84 180)
+		(at 27.94 96.52 180)
 		(fields_autoplaced yes)
 		(effects
@@
 		)
 		(property "Intersheetrefs" "${INTERSHEET_REFS}"
-			(at 20.7204 116.84 0)
+			(at 20.7204 96.52 0)
 			(effects
 				(font
@@
 	(global_label "LTDC_R7"
 		(shape input)
-		(at 27.94 99.06 180)
+		(at 27.94 119.38 180)
 		(fields_autoplaced yes)
 		(effects
@@
 		)
 		(property "Intersheetrefs" "${INTERSHEET_REFS}"
-			(at 20.7204 99.06 0)
+			(at 20.7204 119.38 0)
 			(effects
 				(font
@@
 	(global_label "LTDC_R6"
 		(shape input)
-		(at 27.94 96.52 180)
+		(at 27.94 116.84 180)
 		(fields_autoplaced yes)
 		(effects
@@
 		)
 		(property "Intersheetrefs" "${INTERSHEET_REFS}"
-			(at 20.7204 96.52 0)
+			(at 20.7204 116.84 0)
 			(effects
 				(font
@@
 	(global_label "LTDC_G7"
 		(shape input)
-		(at 27.94 119.38 180)
+		(at 27.94 99.06 180)
 		(fields_autoplaced yes)
 		(effects
@@
 		)
 		(property "Intersheetrefs" "${INTERSHEET_REFS}"
-			(at 20.7204 119.38 0)
+			(at 20.7204 99.06 0)
 			(effects
 				(font
@@
 	(global_label "LTDC_G4"
 		(shape input)
-		(at 27.94 111.76 180)
+		(at 27.94 91.44 180)
 		(fields_autoplaced yes)
 		(effects
@@
 		)
 		(property "Intersheetrefs" "${INTERSHEET_REFS}"
-			(at 20.7204 111.76 0)
+			(at 20.7204 91.44 0)
 			(effects
 				(font
@@
 	(global_label "LTDC_G5"
 		(shape input)
-		(at 27.94 114.3 180)
+		(at 27.94 93.98 180)
 		(fields_autoplaced yes)
 		(effects
@@
 		)
 		(property "Intersheetrefs" "${INTERSHEET_REFS}"
-			(at 20.7204 114.3 0)
+			(at 20.7204 93.98 0)
 			(effects
 				(font

Commit message: #7
Parts:
- added C72, C73: 100n, PCM_EEZ_passives:C_0402_1005Metric, symbol PCM_EEZ_passives:C-EU
- added IC10: LSF0102DCH, PCM_EEZ_SMD:U_SOT765-1_NEX-L, symbol PCM_EEZ_ICs:LSF0102DCH
- renumbered C72 to C74, C73 to C75, C74 to C76, C75 to C77, C76 to C78, C77 to C79, IC10 to IC11
Connections:
- net +3V3: now also C72.2, IC10.2 (REFA), IC10.8 (EN)
- net GND: now also C72.1, C73.1, IC10.1 (GND)
- net REAR_DVID_SCL: now also IC10.6 (B1); no longer IC9.40 (SCL_B)
- net REAR_DVID_SDA: now also IC10.5 (B2); no longer IC9.39 (SDA_B)
- new net: IC10.4 (A2), IC9.39 (SDA_B)
- new net: IC10.3 (A1), IC9.40 (SCL_B)
- new net +5V: C73.2, IC10.7 (REFB)
Other:
- moved on the sheet: C70, IC9

Commit message: #8
Parts:
- added R23, R24: 1K5, PCM_EEZ_passives:R_0402_1005Metric, symbol PCM_EEZ_passives:R-EU
- IC10: value LSF0102DCH -> LSF0204GU12; footprint PCM_EEZ_SMD:U_SOT765-1_NEX-L -> PCM_EEZ_SMD:XQFN12_SOT1174-1_NEX-L; symbol PCM_EEZ_ICs:LSF0102DCH -> PCM_EEZ_ICs:LSF0204GU12; TME LSF0102DCH -> -
- renumbered R23 to R25
Connections:
- net +3V3: now also IC10.1 (Vref_A), IC10.12 (EN); no longer IC10.2 (REFA), IC10.8 (EN)
- net +5V: now also IC10.11 (Vref_B), R23.2, R24.2; no longer IC10.7 (REFB)
- net GND: now also IC10.6 (GND); no longer IC10.1 (GND)
- net REAR_DVID_CEC: now also IC10.7 (B4); no longer IC9.20 (CEC_B)
- net REAR_DVID_HPD: now also IC10.8 (B3); no longer IC9.21 (HPD_B)
- net REAR_DVID_SCL: now also IC10.10 (B1), R23.1; no longer IC10.6 (B1)
- net REAR_DVID_SDA: now also IC10.9 (B2), R24.1; no longer IC10.5 (B2)
- net at IC10.4 (A3): now also IC9.21 (HPD_B); no longer IC9.39 (SDA_B)
- net at IC10.3 (A2): now also IC9.39 (SDA_B); no longer IC9.40 (SCL_B)
- new net: IC10.5 (A4), IC9.20 (CEC_B)
- new net: IC10.2 (A1), IC9.40 (SCL_B)
Other:
- moved on the sheet: C72, C73
