File: KiCad/Ethernet_flash.kicad_sch (KiCad schematic)
At the start: 35 parts, among them IC10 LSF0204GU12, IC11 MX25UM25645GXDI00-T, IC8 TFP410PAP, IC9 TS3DV642A0RUAR

Commit message: #9
Parts:
- added R22: 10K, PCM_EEZ_passives:R_0402_1005Metric, symbol PCM_EEZ_passives:R-EU
- IC11: renamed from IC10; DigiKey 1727-LSF0102DCHCT-ND -> 1727-LSF0204GU12-Q100XTR-ND; LCSC C4363955 -> C7296193; Mouser 771-LSF0102DCH -> 771-LSF0204GU12Q100X
- renumbered C61 to C62, C62 to C63, C63 to C64, C64 to C65, C65 to C66, C66 to C67, C67 to C68, C68 to C69, C69 to C70, C70 to C71, C71 to C72, C72 to C73, C73 to C74, C74 to C75, C75 to C76, C76 to C77, C77 to C78, C78 to C79, C79 to C80, IC9 to IC10, IC11 to IC12, IC8 to IC9, JP2 to JP1, R22 to R23, R23 to R24, R24 to R25, R25 to R26
Connections:
- net +3V3: now also R22.2
- net at IC10.21 (HPD_B), IC11.4 (A3): now also R22.1
Other:
- moved on the sheet: C73, C74, IC11, R24, R25

Commit message: #10
Connections:
- net GND: now also IC9.34 (RESERVED)
Changed lines of the file:
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@@
 	(title_block
 		(title "${project_name}")
-		(date "2025-12-28")
+		(date "2025-12-30")
 		(rev "${project_version}")
 		(company "${project_creator}")
@@
 	)
 	(junction
+		(at 66.04 83.82)
+		(diameter 0)
+		(color 0 0 0 0)
+	)
+	(junction
 		(at 73.66 132.08)
 		(diameter 0)
@@
 		)
 		(stroke
+			(width 0)
+			(type default)
+		)
+	)
+	(wire
+		(pts
+			(xy 60.96 83.82) (xy 66.04 83.82)
+		)
+		(stroke

Commit message: #12
Parts:
- renumbered C62 to C63, C63 to C64, C64 to C65, C65 to C66, C66 to C67, C67 to C68, C68 to C69, C69 to C70, C70 to C71, C71 to C72, C72 to C73, C73 to C74, C74 to C75, C75 to C76, C76 to C77, C77 to C78, C78 to C79, C79 to C80, C80 to C81, R18 to R20, R19 to R21, R20 to R22, R21 to R23, R22 to R24, R23 to R25, R24 to R26, R25 to R27, R26 to R28
