File: KiCad/eth_psram_emmc.kicad_sch (KiCad schematic)
At the start: 39 parts, among them IC5 MX52LM04A11XVW, IC6 LAN8742A-CZ-TR, IC7 APS256XXN-OBR-BG, Y2 VXM7-9032-25M0000000

Commit message: #4
Parts:
- removed IC5: MX52LM04A11XVW, PCM_EEZ_BGA:BGA153_MX52LM_EMMC, symbol PCM_EEZ_ICs:MX52LM04A11XVW
- added IC5: IS21EF04GP-JQLI, PCM_EEZ_BGA:IS21EF04GP-JQLI, symbol PCM_EEZ_ICs:IS21EF04GP-JQLI
- renumbered R9 to R10, R10 to R11, R11 to R12, R12 to R13, R13 to R14, R14 to R15, R15 to R16, R16 to R17, R4 to R5, R5 to R6, R6 to R7, R7 to R8, R8 to R9
Connections:
- net +1V8: now also IC5.H3 (VCCQ), IC5.H8 (VCCQ), IC5.L2 (VCCQ), IC5.L4 (VCCQ), IC5.L7 (VCCQ), IC5.L9 (VCCQ), IC5.M7 (VCCQ), IC5.P3 (VCCQ), IC5.P8 (VCCQ)
- net +3V3: now also IC5.F2 (VCC), IC5.F3 (VCC), IC5.F4 (VCC), IC5.F5 (VCC), IC5.F6 (VCC), IC5.F7 (VCC), IC5.F8 (VCC), IC5.F9 (VCC)
- net GND: now also IC5.G2 (VSS), IC5.G3 (VSS), IC5.G4 (VSS), IC5.G5 (VSS), IC5.G6 (VSS), IC5.G7 (VSS), IC5.G8 (VSS), IC5.G9 (VSS), IC5.H2 (VSSQ), IC5.H9 (VSSQ), IC5.J5 (VSS), IC5.L3 (VSSQ), IC5.L8 (VSSQ), IC5.M4 (VSSQ), IC5.P2 (VSSQ), IC5.P9 (VSSQ)
- net SDMMC_CLK: now also IC5.P6 (CLK)
- net SDMMC_CMD: now also IC5.P5 (CMD)
- net SDMMC_D0: now also IC5.K2 (DAT0)
- net SDMMC_D1: now also IC5.N2 (DAT1)
- net SDMMC_D2: now also IC5.K3 (DAT2)
- net SDMMC_D3: now also IC5.N3 (DAT3)
- net SDMMC_D4: now also IC5.N8 (DAT4)
- net SDMMC_D5: now also IC5.K8 (DAT5)
- net SDMMC_D6: now also IC5.N9 (DAT6)
- net SDMMC_D7: now also IC5.K9 (DAT7)
- net ~{RESET_OUT}: now also IC5.M5 (RST_N)
- net at C46.1, C49.1: now also IC5.E4 (VDDI)
Other:
- moved on the sheet: C44, C46, C47, C49

Commit message: #9
Parts:
- renumbered C42 to C43, C43 to C44, C44 to C45, C45 to C46, C46 to C47, C47 to C48, C48 to C49, C49 to C50, C50 to C51, C51 to C52, C52 to C53, C53 to C54, C54 to C55, C55 to C56, C56 to C57, C57 to C58, C58 to C59, C59 to C60, C60 to C61, IC5 to IC6, IC6 to IC7, IC7 to IC8
