File: KiCad/eth_psram_emmc.kicad_sch (KiCad schematic)
At the start: 39 parts, among them IC6 IS21EF04GP-JQLI, IC7 LAN8742A-CZ-TR, IC8 APS256XXN-OBR-BG, Y2 VXM7-9032-25M0000000

Commit message: #12
Parts:
- added C51: 10n, PCM_EEZ_passives:C_0402_1005Metric, symbol PCM_EEZ_passives:C-EU
- added R14, R19: 220R, PCM_EEZ_passives:R_0402_1005Metric, symbol PCM_EEZ_passives:R-EU
- R12: now not fitted; now left out of the parts list
- renumbered C51 to C52, C52 to C53, C53 to C54, C54 to C55, C55 to C56, C56 to C57, C57 to C58, C58 to C59, C59 to C60, C60 to C61, C61 to C62, R14 to R15, R15 to R16, R16 to R17, R17 to R18
Connections:
- net +3V3: now also C51.1
- net GND: now also C51.2
- net ~{ETH_LINK100}: now also R19.2; no longer IC7.2 (LED2/NINT/NPME/NINTSEL), R11.1
- net ~{ETH_LINK_ACT}: now also R14.2; no longer IC7.3 (LED1/NINT/NPME/REGOFF), R12.2
- new net: IC7.2 (LED2/NINT/NPME/NINTSEL), R11.1, R19.1
- new net: IC7.3 (LED1/NINT/NPME/REGOFF), R12.2, R14.1
Other:
- moved on the sheet: C43, C44, C52, C53, C54, C55, C56, C57, C58, FB2, IC7, R10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

Commit message: Eth PHY straps updated
Connections:
- net ETH_RX_ERR: now also R12.1
- net GND: now also R12.2; no longer R12.1
- net at IC7.3 (LED1/NINT/NPME/REGOFF), R14.1: no longer R12.2
Other:
- moved on the sheet: R12, R5, R6, R7, R9, RN1A, RN1B, RN1C, RN1D, RN2A, RN2B, RN2C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

Commit message: Schematics update
Other:
- note added: "PA2"
- note added: "PA7"
- note added: "PB10"
- note added: "PB7"
- note added: "PC1"
- note added: "PC4"
- note added: "PC5"
- note added: "PD7"
- note added: "PG11"
- note added: "PG13"
Changed lines of the file:
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@@
 		(comment 3 "${project_url}")
 	)
+	(text "PD7"
+		(exclude_from_sim no)
+		(at 27.94 66.04 0)
+		(effects
+			(font
+				(size 0.889 0.889)
+				(color 132 0 132 1)
+			)
+			(justify left bottom)
+		)
+	)
+	(text "PG11"
+		(exclude_from_sim no)
+		(at 27.94 33.02 0)
+		(effects
+			(font
+				(size 0.889 0.889)
+				(color 132 0 132 1)
+			)
+			(justify left bottom)
+		)
+	)
 	(text "TD matched Net Lengths [Tolerance = 100mil]\nDiff Pair 100ohm"
 		(exclude_from_sim no)
@@
 		)
 	)
+	(text "PG13"
+		(exclude_from_sim no)
+		(at 27.94 35.56 0)
+		(effects
+			(font
+				(size 0.889 0.889)
+				(color 132 0 132 1)
+			)
+			(justify left bottom)
+		)
+	)
+	(text "PA7"
+		(exclude_from_sim no)
+		(at 27.94 53.34 0)
+		(effects
+			(font
+				(size 0.889 0.889)
+				(color 132 0 132 1)
+			)
+			(justify left bottom)
+		)
+	)
+	(text "PB10"
+		(exclude_from_sim no)
+		(at 27.94 48.26 0)
+		(effects
+			(font
+				(size 0.889 0.889)
+				(color 132 0 132 1)
+			)
+			(justify left bottom)
+		)
+	)
 	(text "PSRAM 256 Mbit"
 		(exclude_from_sim no)
@@
 		)
 	)
+	(text "PC4"
+		(exclude_from_sim no)
+		(at 27.94 43.18 0)
+		(effects
+			(font
+				(size 0.889 0.889)
+				(color 132 0 132 1)
+			)
+			(justify left bottom)
+		)
+	)
+	(text "PB7"
+		(exclude_from_sim no)
+		(at 27.94 38.1 0)
+		(effects
+			(font
+				(size 0.889 0.889)
+				(color 132 0 132 1)
+			)
+			(justify left bottom)
+		)
+	)
+	(text "PA2"
+		(exclude_from_sim no)
+		(at 27.94 58.42 0)
+		(effects
+			(font
+				(size 0.889 0.889)
+				(color 132 0 132 1)
+			)
+			(justify left bottom)
+		)
+	)
 	(text "Ethernet RMII PHY"
 		(exclude_from_sim no)
@@
 		)
 	)
+	(text "PC5"
+		(exclude_from_sim no)
+		(at 27.94 45.72 0)
+		(effects
+			(font
+				(size 0.889 0.889)
+				(color 132 0 132 1)
+			)
+			(justify left bottom)
+		)
+	)
+	(text "PC1"
+		(exclude_from_sim no)
+		(at 27.94 55.88 0)
+		(effects
+			(font
+				(size 0.889 0.889)
+				(color 132 0 132 1)
+			)
+			(justify left bottom)
+		)
+	)
 	(text_box "HEXASPI Impedance Constraint: Min = 45.00, Max = 55.00"
 		(exclude_from_sim no)
@@
 	(wire
 		(pts
-			(xy 30.48 53.34) (xy 35.56 53.34)
+			(xy 25.4 53.34) (xy 35.56 53.34)
 		)
 		(stroke
@@
 	(wire
 		(pts
-			(xy 30.48 58.42) (xy 35.56 58.42)
+			(xy 25.4 58.42) (xy 35.56 58.42)
 		)
 		(stroke
@@
 	(wire
 		(pts
-			(xy 30.48 33.02) (xy 81.28 33.02)
+			(xy 25.4 33.02) (xy 81.28 33.02)
 		)
 		(stroke
@@
 	(wire
 		(pts
-			(xy 30.48 45.72) (xy 35.56 45.72)
+			(xy 25.4 45.72) (xy 35.56 45.72)
 		)
 		(stroke
@@
 	(wire
 		(pts
-			(xy 30.48 55.88) (xy 35.56 55.88)
+			(xy 25.4 55.88) (xy 35.56 55.88)
 		)
 		(stroke
@@
 	(wire
 		(pts
-			(xy 30.48 48.26) (xy 60.96 48.26)
+			(xy 25.4 48.26) (xy 60.96 48.26)
 		)
 		(stroke
@@
 	(wire
 		(pts
-			(xy 30.48 43.18) (xy 35.56 43.18)
+			(xy 25.4 43.18) (xy 35.56 43.18)
 		)
 		(stroke
@@
 	(wire
 		(pts
-			(xy 30.48 35.56) (xy 35.56 35.56)
+			(xy 25.4 35.56) (xy 35.56 35.56)
 		)
 		(stroke
@@
 	(wire
 		(pts
-			(xy 30.48 66.04) (xy 35.56 66.04)
+			(xy 25.4 66.04) (xy 35.56 66.04)
 		)
 		(stroke
@@
 	(wire
 		(pts
-			(xy 30.48 63.5) (xy 81.28 63.5)
+			(xy 25.4 63.5) (xy 81.28 63.5)
 		)
 		(stroke
@@
 	(wire
 		(pts
-			(xy 30.48 38.1) (xy 35.56 38.1)
+			(xy 25.4 38.1) (xy 35.56 38.1)
 		)
 		(stroke
@@
 	(global_label "~{RESET_OUT}"
 		(shape input)
-		(at 30.48 63.5 180)
+		(at 25.4 63.5 180)
 		(fields_autoplaced yes)
 		(effects
@@
 		)
 		(property "Intersheetrefs" "${INTERSHEET_REFS}"
-			(at 21.6096 63.5 0)
+			(at 16.5296 63.5 0)
 			(effects
 				(font
@@
 	(global_label "ETH_RX_ERR"
 		(shape output)
-		(at 30.48 48.26 180)
+		(at 25.4 48.26 180)
 		(fields_autoplaced yes)
 		(effects
@@
 		)
 		(property "Intersheetrefs" "${INTERSHEET_REFS}"
-			(at 20.7629 48.26 0)
+			(at 15.6829 48.26 0)
 			(effects
 				(font
@@
 	(global_label "ETH_REF_CLK"
 		(shape output)
-		(at 30.48 66.04 180)
+		(at 25.4 66.04 180)
 		(fields_autoplaced yes)
 		(effects
@@
 		)
 		(property "Intersheetrefs" "${INTERSHEET_REFS}"
-			(at 20.1279 66.04 0)
+			(at 15.0479 66.04 0)
 			(effects
 				(font
@@
 	(global_label "ETH_TX_EN"
 		(shape input)
-		(at 30.48 33.02 180)
+		(at 25.4 33.02 180)
 		(fields_autoplaced yes)
 		(effects
@@
 		)
 		(property "Intersheetrefs" "${INTERSHEET_REFS}"
-			(at 21.8213 33.02 0)
+			(at 16.7413 33.02 0)
 			(effects
 				(font
@@
 	(global_label "ETH_RXD0"
 		(shape output)
-		(at 30.48 43.18 180)
+		(at 25.4 43.18 180)
 		(fields_autoplaced yes)
 		(effects
@@
 		)
 		(property "Intersheetrefs" "${INTERSHEET_REFS}"
-			(at 22.2868 43.18 0)
+			(at 17.2068 43.18 0)
 			(effects
 				(font
@@
 	(global_label "ETH_RXD1"
 		(shape output)
-		(at 30.48 45.72 180)
+		(at 25.4 45.72 180)
 		(fields_autoplaced yes)
 		(effects
@@
 		)
 		(property "Intersheetrefs" "${INTERSHEET_REFS}"
-			(at 22.2868 45.72 0)
+			(at 17.2068 45.72 0)
 			(effects
 				(font
@@
 	(global_label "ETH_MDC"
 		(shape input)
-		(at 30.48 55.88 180)
+		(at 25.4 55.88 180)
 		(fields_autoplaced yes)
 		(effects
@@
 		)
 		(property "Intersheetrefs" "${INTERSHEET_REFS}"
-			(at 22.9642 55.88 0)
+			(at 17.8842 55.88 0)
 			(effects
 				(font
@@
 	(global_label "ETH_MDIO"
 		(shape bidirectional)
-		(at 30.48 58.42 180)
+		(at 25.4 58.42 180)
 		(fields_autoplaced yes)
 		(effects
@@
 		)
 		(property "Intersheetrefs" "${INTERSHEET_REFS}"
-			(at 21.8318 58.42 0)
+			(at 16.7518 58.42 0)
 			(effects
 				(font
@@
 	(global_label "ETH_TXD0"
 		(shape input)
-		(at 30.48 35.56 180)
+		(at 25.4 35.56 180)
 		(fields_autoplaced yes)
 		(effects
@@
 		)
 		(property "Intersheetrefs" "${INTERSHEET_REFS}"
-			(at 22.4985 35.56 0)
+			(at 17.4185 35.56 0)
 			(effects
 				(font
@@
 	(global_label "ETH_CRS_DV"
 		(shape output)
-		(at 30.48 53.34 180)
+		(at 25.4 53.34 180)
 		(fields_autoplaced yes)
 		(effects
@@
 		)
 		(property "Intersheetrefs" "${INTERSHEET_REFS}"
-			(at 20.8052 53.34 0)
+			(at 15.7252 53.34 0)
 			(effects
 				(font
@@
 	(global_label "ETH_TXD1"
 		(shape input)
-		(at 30.48 38.1 180)
+		(at 25.4 38.1 180)
 		(fields_autoplaced yes)
 		(effects
@@
 		)
 		(property "Intersheetrefs" "${INTERSHEET_REFS}"
-			(at 22.4985 38.1 0)
+			(at 17.4185 38.1 0)
 			(effects
 				(font
